File: 1-BAGEL.kicad_sch (KiCad schematic)
At the start: 32 parts, among them J1 Conn_01x06_Male, Q1 QPNP, U1 HX711, U2 MAX31856

Commit message: schematic draft
Connections:
- net 3V_OUT: no longer C3.1, Q1.3 (E)
- net 5V_OUT: now also C3.1, Q1.3 (E)
Changed lines of the file:
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@@
     (effects (font (size 1.27 1.27)) (justify right bottom))
   )
-  (label "3V_OUT" (at 114.3 30.48 180)
+  (label "5V_OUT" (at 114.3 30.48 180)
     (effects (font (size 1.27 1.27)) (justify right bottom))
   )
